Commit message: update pkg

File: catkin_ws/src/robot/vx300s/interbotix_ros_manipulators/interbotix_ros_xsarms/interbotix_xsarm_descriptions/urdf/vx300s.urdf.xacro (robot description, xacro)
@@ -9,5 +9,7 @@
   <xacro:arg name="external_urdf_loc" default=""/>
   <xacro:arg name="load_gazebo_configs" default="false"/>
+  <xacro:arg name="wrist_rotation_length" default="0.0"/>
   <xacro:property name="urdf_loc" value="$(arg external_urdf_loc)"/>
+  <xacro:property name="rotation_length" value="$(arg wrist_rotation_length)"/>
   <xacro:property name="pi_offset" value="0.00001"/>
   <xacro:if value="$(arg load_gazebo_configs)">
@@ -232,5 +234,5 @@
     <axis xyz="1 0 0"/>
     <limit effort="1" lower="${-pi + pi_offset}" upper="${pi - pi_offset}" velocity="${pi}"/>
-    <origin rpy="0 0 0" xyz="0.069744 0 0"/>
+    <origin rpy="0 0 0" xyz="${0.069744 + rotation_length} 0 0"/>
     <parent link="$(arg robot_name)/wrist_link"/>
     <child link="$(arg robot_name)/gripper_link"/>
